Commit message: Implementation of PI controller and changed the robot model to fix stability issues

File: src/my_robot/urdf/new_robot.xacro (robot description, xacro)
@@ -58,5 +58,5 @@
     <link name='chassis'>
 		<inertial>
-			<mass value="3.0"/>
+			<mass value="8.0"/>
 		  	<origin xyz="0 0 0" rpy=" 0 0 0"/>
 		  	<inertia
@@ -68,5 +68,5 @@
 		  	<origin xyz="0 0 0" rpy=" 0 0 -1.5707"/>
 		  	<geometry>
-		    	<box size="0.45 0.45 .1"/>
+		    	<box size="0.5 0.5 .1"/>
 		  	</geometry>
 		</collision>
@@ -74,5 +74,5 @@
 		  	<origin xyz="0 0 0" rpy=" 0 0 -1.5707"/>
 		  	<geometry>
-		    	<box size="0.45 0.45 .1"/>
+		    	<box size="0.5 0.5 .1"/>
 			</geometry>
 		</visual>
@@ -90,11 +90,11 @@
 			<origin xyz="0 0 0" rpy="1.5707 0 0"/>
 			<geometry>
-				<cylinder radius="0.06" length="0.05"/>
-			</geometry>
-		</visual>
-		<collision>
-			<origin xyz="0 0 0" rpy="1.5707 0 0"/>
-			<geometry>
-				<cylinder radius="0.06" length="0.05"/>
+				<cylinder radius="0.1" length="0.05"/>
+			</geometry>
+		</visual>
+		<collision>
+			<origin xyz="0 0 0" rpy="1.5707 0 0"/>
+			<geometry>
+				<cylinder radius="0.1" length="0.05"/>
 			</geometry>
 		</collision>
@@ -112,11 +112,11 @@
 			<origin xyz="0 0 0" rpy="1.5707 0 0"/>
 			<geometry>
-				<cylinder radius="0.06" length="0.05"/>
-			</geometry>
-		</visual>
-		<collision>
-			<origin xyz="0 0 0" rpy="1.5707 0 0"/>
-			<geometry>
-				<cylinder radius="0.06" length="0.05"/>
+				<cylinder radius="0.1" length="0.05"/>
+			</geometry>
+		</visual>
+		<collision>
+			<origin xyz="0 0 0" rpy="1.5707 0 0"/>
+			<geometry>
+				<cylinder radius="0.1" length="0.05"/>
 			</geometry>
 		</collision>
@@ -134,11 +134,11 @@
 			<origin xyz="0 0 0" rpy="1.5707 0 0"/>
 			<geometry>
-				<cylinder radius="0.06" length="0.05"/>
-			</geometry>
-		</visual>
-		<collision>
-			<origin xyz="0 0 0" rpy="1.5707 0 0"/>
-			<geometry>
-				<cylinder radius="0.06" length="0.05"/>
+				<cylinder radius="0.1" length="0.05"/>
+			</geometry>
+		</visual>
+		<collision>
+			<origin xyz="0 0 0" rpy="1.5707 0 0"/>
+			<geometry>
+				<cylinder radius="0.1" length="0.05"/>
 			</geometry>
 		</collision>
@@ -156,11 +156,11 @@
 			<origin xyz="0 0 0" rpy="1.5707 0 0"/>
 			<geometry>
-				<cylinder radius="0.06" length="0.05"/>
-			</geometry>
-		</visual>
-		<collision>
-			<origin xyz="0 0 0" rpy="1.5707 0 0"/>
-			<geometry>
-				<cylinder radius="0.06" length="0.05"/>
+				<cylinder radius="0.1" length="0.05"/>
+			</geometry>
+		</visual>
+		<collision>
+			<origin xyz="0 0 0" rpy="1.5707 0 0"/>
+			<geometry>
+				<cylinder radius="0.1" length="0.05"/>
 			</geometry>
 		</collision>
@@ -168,5 +168,5 @@
     <link name='tower'>
 		<inertial>
-			<mass value="0.1"/>
+			<mass value="1"/>
 			<origin xyz="0.0 0 0" rpy=" 0 0 0"/>
 			<inertia
@@ -178,5 +178,5 @@
 			<origin xyz="0 0 0" rpy="0 0 0"/>
 			<geometry>
-				<cylinder radius="0.21" length="0.2"/>
+				<cylinder radius="0.22" length="0.12"/>
 			</geometry>
 		</visual>
@@ -184,42 +184,15 @@
 			<origin xyz="0 0 0" rpy="0 0 0"/>
 			<geometry>
-				<cylinder radius="0.21" length="0.2"/>
-			</geometry>
-		</collision>
-	</link>
-	<link name='cap'>
-		<inertial>
-			<mass value="0.1"/>
-		  	<origin xyz="0 0 0" rpy=" 0 1.5707 1.5707"/>
-		  	<inertia
-		      ixx="0.1" ixy="0" ixz="0"
-		      iyy="0.1" iyz="0"
-		      izz="0.1"/>
-		</inertial>
-		<collision>
-			<origin xyz="0 0 0" rpy=" 0 0 0"/>
-		  	<geometry>
-		    	<sphere radius="0.209"/>
-		  	</geometry>
-		</collision>
-		<visual>
-			<origin xyz="0 0 0" rpy=" 0 0 0"/>
-			<geometry>
-		    	<sphere radius="0.209"/>
-		  	</geometry>
-		</visual>
-	</link>
-	<joint name="tower_cap" type="fixed">
-		<origin xyz="0 0 0.09" rpy="0 0 0" />
-		<parent link="tower"/>
-		<child link="cap" />
-	</joint>
+				<cylinder radius="0.22" length="0.12"/>
+			</geometry>
+		</collision>
+	</link>
 	<joint name="chassis_tower" type="fixed">
-		<origin xyz="0 0 0.14" rpy="0 0 0" />
+		<origin xyz="0 0 0.10" rpy="0 0 0" />
 		<parent link="chassis"/>
 		<child link="tower" />
 	</joint>
 	<joint name="left_front_axis" type="continuous">
-		<origin xyz="0.16 0.2505 -0.02" rpy="0 0 0"/>
+		<origin xyz="0.2 0.278 0.02" rpy="0 0 0"/>
 		<child link="wheel_left_front"/>
 		<parent link="chassis"/>
@@ -229,5 +202,5 @@
 	</joint>
 	<joint name="left_back_axis" type="continuous">
-		<origin xyz="-0.16 0.2505 -0.02" rpy="0 0 0"/>
+		<origin xyz="-0.2 0.278 0.02" rpy="0 0 0"/>
 		<child link="wheel_left_back"/>
 		<parent link="chassis"/>
@@ -237,5 +210,5 @@
 	</joint>
 	<joint name="right_back_axis" type="continuous">
-		<origin xyz="-0.16 -0.2505 -0.02" rpy="0 0 0"/>
+		<origin xyz="-0.2 -0.278 0.02" rpy="0 0 0"/>
 		<child link="wheel_right_back"/>
 		<parent link="chassis"/>
@@ -245,5 +218,5 @@
 	</joint>
 	<joint name="right_front_axis" type="continuous">
-		<origin xyz="0.16 -0.2505 -0.02" rpy="0 0 0"/>
+		<origin xyz="0.2 -0.278 0.02" rpy="0 0 0"/>
 		<child link="wheel_right_front"/>
 		<parent link="chassis"/>
@@ -275,5 +248,5 @@
 	</link>
   <joint type="fixed" name="hokuyo_joint">
-    <origin xyz="0 0 0.32" rpy="0 0 0"/>
+    <origin xyz="0 0 0.08" rpy="0 0 0"/>
     <child link="hokuyo"/>
     <parent link="tower"/>
@@ -303,5 +276,5 @@
 	</link>
   <joint type="fixed" name="camera_joint">
-    <origin xyz="0.215 0 -0.03" rpy="0 0 0"/>
+    <origin xyz="0.265 0 -0.03" rpy="0 0 0"/>
     <child link="camera"/>
     <parent link="chassis"/>

Commit message: Where Am I project submission

File: src/my_robot/urdf/new_robot.xacro (robot description, xacro)
@@ -68,5 +68,5 @@
 		  	<origin xyz="0 0 0" rpy=" 0 0 -1.5707"/>
 		  	<geometry>
-		    	<box size="0.5 0.5 .1"/>
+		    	<box size="0.6 0.6 .1"/>
 		  	</geometry>
 		</collision>
